File: Communication.sch (KiCad schematic (older format))
At the start: 58 parts, among them IC1 LAN8720, IC2 USB2514B, IC3 MAX3221, IC4 TPS2033, IC5 WE-TVS-82400274, IC6 WE-TVS-82400274, Y1 24M,18p

Commit message: LILY notitzen hinzugefügt
Other:
- note added: "LILY-W1 series \nHost-based Wi-Fi modules"
- note added: "NEO-M8 \nu-blox M8 concurrent GNSS modules"
Changed lines of the file:
@@
 F7 "USB_D-" I L 800 1300 60
 $EndSheet
-Text Notes 750  2300 0    60   ~ 0
+Text Notes 800  2300 0    60   ~ 0
 TOBY-L2 series \nLTE/DC-HSPA+/EGPRS modules \n
 $Sheet
@@
 F1 "NEO.sch" 60
 $EndSheet
+Text Notes 850  3800 0    60   ~ 0
+LILY-W1 series \nHost-based Wi-Fi modules
+Text Notes 2400 2300 0    60   ~ 0
+NEO-M8 \nu-blox M8 concurrent GNSS modules
 $EndSCHEMATC

Commit message: added footprintadded footprintss
Parts:
- removed C1, C12, C13, C14, C15: 22u,10V, Passives:C1206N, symbol C
- removed C10, C11, C2, C3, C4, C5, C8, C9: 100n, Passives:C0402N, symbol C
- removed C6, C7: 18p, Passives:C0402N, symbol C
- removed IC2: USB2514B, USB_IC:USB251xB_QFN36, symbol USB251xB
- removed IC4: TPS2033, USB_IC:TPS203xD, symbol TPS203x
- removed IC5, IC6: WE-TVS-82400274, USB_IC:WE-TVS-82400274_SC70, symbol WE-TVS-82400274
- removed R1, R2, R3, R4: 100k, Passives:R0402N, symbol R
- removed R5: 12k, Passives:R0402N, symbol R
- removed R6: 10k, Passives:R0402N, symbol R
- removed Y1: 24M,18p, Crystals:Crystal_3.2x2.5, symbol Crystal4

Commit message: NEO_modifiziert
Parts:
- removed C27, C28, C29, C30, C31: 100n,16V, Passives:C0402N, symbol C
- removed C39: 22u,10V, Passives:C1206N, symbol C
- removed IC3: MAX3221, Communication:MAX3221_TSSOP, symbol MAX3221
- removed R22: 22R, Passives:R0402N, symbol R
