File: TOBY.sch (KiCad schematic (older format))
At the start: 36 parts, among them Q301 2N7002BKT, U301 U-BLOX-TOBY-L2, X301 ANT, X302 SIMcard, X303 ANT

Commit message: sorted components
Parts:
- R304: value R -> 0
Other:
- note added: "So groß?"
Changed lines of the file:
@@
 $EndComp
 $Comp
-L GND #PWR084
+L GND #PWR321
 U 1 1 570E3CB9
 P 9100 2450
-F 0 "#PWR084" H 9100 2200 50  0001 C CNN
+F 0 "#PWR321" H 9100 2200 50  0001 C CNN
 F 1 "GND" H 9100 2300 50  0000 C CNN
 F 2 "" H 9100 2450 50  0000 C CNN
@@
 $EndComp
 $Comp
-L GND #PWR085
+L GND #PWR322
 U 1 1 570E6A84
 P 10000 5500
-F 0 "#PWR085" H 10000 5250 50  0001 C CNN
+F 0 "#PWR322" H 10000 5250 50  0001 C CNN
 F 1 "GND" H 10000 5350 50  0000 C CNN
 F 2 "" H 10000 5500 50  0000 C CNN
@@
 $EndComp
 $Comp
-L GND #PWR086
+L GND #PWR319
 U 1 1 570F627C
 P 8550 5950
-F 0 "#PWR086" H 8550 5700 50  0001 C CNN
+F 0 "#PWR319" H 8550 5700 50  0001 C CNN
 F 1 "GND" H 8550 5800 50  0000 C CNN
 F 2 "" H 8550 5950 50  0000 C CNN
@@
 NoConn ~ 5600 5500
 $Comp
-L GND #PWR087
+L GND #PWR309
 U 1 1 570F7F5B
 P 5950 5600
-F 0 "#PWR087" H 5950 5350 50  0001 C CNN
+F 0 "#PWR309" H 5950 5350 50  0001 C CNN
 F 1 "GND" H 5950 5450 50  0000 C CNN
 F 2 "" H 5950 5600 50  0000 C CNN
@@
 $EndComp
 $Comp
-L GND #PWR088
+L GND #PWR308
 U 1 1 570F7F96
 P 4050 5350
-F 0 "#PWR088" H 4050 5100 50  0001 C CNN
+F 0 "#PWR308" H 4050 5100 50  0001 C CNN
 F 1 "GND" H 4050 5200 50  0000 C CNN
 F 2 "" H 4050 5350 50  0000 C CNN
@@
 $EndComp
 $Comp
-L GND #PWR089
+L GND #PWR302
 U 1 1 570FA2F8
 P 1150 2550
-F 0 "#PWR089" H 1150 2300 50  0001 C CNN
+F 0 "#PWR302" H 1150 2300 50  0001 C CNN
 F 1 "GND" H 1150 2400 50  0000 C CNN
 F 2 "" H 1150 2550 50  0000 C CNN
@@
 $EndComp
 $Comp
-L GND #PWR090
+L GND #PWR305
 U 1 1 570FD240
 P 3000 2850
-F 0 "#PWR090" H 3000 2600 50  0001 C CNN
+F 0 "#PWR305" H 3000 2600 50  0001 C CNN
 F 1 "GND" H 3000 2700 50  0000 C CNN
 F 2 "" H 3000 2850 50  0000 C CNN
@@
 $EndComp
 $Comp
-L GND #PWR091
+L GND #PWR318
 U 1 1 571026BC
 P 8500 2800
-F 0 "#PWR091" H 8500 2550 50  0001 C CNN
+F 0 "#PWR318" H 8500 2550 50  0001 C CNN
 F 1 "GND" H 8500 2650 50  0000 C CNN
 F 2 "" H 8500 2800 50  0000 C CNN
@@
 $EndComp
 $Comp
-L GND #PWR092
+L GND #PWR316
 U 1 1 57102715
 P 8200 2800
-F 0 "#PWR092" H 8200 2550 50  0001 C CNN
+F 0 "#PWR316" H 8200 2550 50  0001 C CNN
 F 1 "GND" H 8200 2650 50  0000 C CNN
 F 2 "" H 8200 2800 50  0000 C CNN
@@
 $EndComp
 $Comp
-L GND #PWR093
+L GND #PWR314
 U 1 1 5710276E
 P 7900 2800
-F 0 "#PWR093" H 7900 2550 50  0001 C CNN
+F 0 "#PWR314" H 7900 2550 50  0001 C CNN
 F 1 "GND" H 7900 2650 50  0000 C CNN
 F 2 "" H 7900 2800 50  0000 C CNN
@@
 $EndComp
 $Comp
-L GND #PWR094
+L GND #PWR312
 U 1 1 571027C7
 P 7600 2800
-F 0 "#PWR094" H 7600 2550 50  0001 C CNN
+F 0 "#PWR312" H 7600 2550 50  0001 C CNN
 F 1 "GND" H 7600 2650 50  0000 C CNN
 F 2 "" H 7600 2800 50  0000 C CNN
@@
 $EndComp
 $Comp
-L GND #PWR095
+L GND #PWR320
 U 1 1 571028B7
 P 8800 2800
-F 0 "#PWR095" H 8800 2550 50  0001 C CNN
+F 0 "#PWR320" H 8800 2550 50  0001 C CNN
 F 1 "GND" H 8800 2650 50  0000 C CNN
 F 2 "" H 8800 2800 50  0000 C CNN
@@
 	2050 4200 2050 4300
 $Comp
-L GND #PWR096
+L GND #PWR304
 U 1 1 57105942
 P 2050 4900
-F 0 "#PWR096" H 2050 4650 50  0001 C CNN
+F 0 "#PWR304" H 2050 4650 50  0001 C CNN
 F 1 "GND" H 2050 4750 50  0000 C CNN
 F 2 "" H 2050 4900 50  0000 C CNN
@@
 $EndComp
 $Comp
-L +3V3 #PWR097
+L +3V3 #PWR303
 U 1 1 57105A00
 P 2050 3200
-F 0 "#PWR097" H 2050 3050 50  0001 C CNN
+F 0 "#PWR303" H 2050 3050 50  0001 C CNN
 F 1 "+3V3" H 2050 3340 50  0000 C CNN
 F 2 "" H 2050 3200 50  0000 C CNN
@@
 P 3450 4050
 F 0 "R304" V 3530 4050 50  0000 C CNN
-F 1 "R" V 3375 4050 50  0000 C CNN
+F 1 "0" V 3375 4050 50  0000 C CNN
 F 2 "Passives:R0402N" V 3380 4050 30  0001 C CNN
 F 3 "" H 3450 4050 30  0000 C CNN
@@
 	3450 3650 3450 3850
 $Comp
-L GND #PWR098
+L GND #PWR306
 U 1 1 5710A931
 P 3200 4350
-F 0 "#PWR098" H 3200 4100 50  0001 C CNN
+F 0 "#PWR306" H 3200 4100 50  0001 C CNN
 F 1 "GND" H 3200 4200 50  0000 C CNN
 F 2 "" H 3200 4350 50  0000 C CNN
@@
 $EndComp
 $Comp
-L GND #PWR099
+L GND #PWR307
 U 1 1 5710A99F
 P 3450 4350
-F 0 "#PWR099" H 3450 4100 50  0001 C CNN
+F 0 "#PWR307" H 3450 4100 50  0001 C CNN
 F 1 "GND" H 3450 4200 50  0000 C CNN
 F 2 "" H 3450 4350 50  0000 C CNN
@@
 NoConn ~ 7150 3150
 $Comp
-L +3V8 #PWR0100
+L +3V8 #PWR301
 U 1 1 57114B92
 P 1150 1500
-F 0 "#PWR0100" H 1150 1350 50  0001 C CNN
+F 0 "#PWR301" H 1150 1350 50  0001 C CNN
 F 1 "+3V8" H 1150 1640 50  0000 C CNN
 F 2 "" H 1150 1500 50  0000 C CNN
@@
 Connection ~ 4000 1750
 $Comp
-L +1V8 #PWR0101
+L +1V8 #PWR310
 U 1 1 57168AFB
 P 7400 1500
-F 0 "#PWR0101" H 7400 1350 50  0001 C CNN
+F 0 "#PWR310" H 7400 1350 50  0001 C CNN
 F 1 "+1V8" H 7400 1640 50  0000 C CNN
 F 2 "" H 7400 1500 50  0000 C CNN
@@
 	7400 1600 7400 1500
 $Comp
-L GND #PWR0102
+L GND #PWR323
 U 1 1 571D4F40
 P 10600 2500
-F 0 "#PWR0102" H 10600 2250 50  0001 C CNN
+F 0 "#PWR323" H 10600 2250 50  0001 C CNN
 F 1 "GND" H 10600 2350 50  0000 C CNN
 F 2 "" H 10600 2500 50  0000 C CNN
@@
 $EndComp
 $Comp
-L GND #PWR0103
+L GND #PWR311
 U 1 1 5723D09C
 P 7600 1000
-F 0 "#PWR0103" H 7600 750 50  0001 C CNN
+F 0 "#PWR311" H 7600 750 50  0001 C CNN
 F 1 "GND" H 7600 850 50  0000 C CNN
 F 2 "" H 7600 1000 50  0000 C CNN
@@
 $EndComp
 $Comp
-L GND #PWR0104
+L GND #PWR313
 U 1 1 5723D15B
 P 7900 1000
-F 0 "#PWR0104" H 7900 750 50  0001 C CNN
+F 0 "#PWR313" H 7900 750 50  0001 C CNN
 F 1 "GND" H 7900 850 50  0000 C CNN
 F 2 "" H 7900 1000 50  0000 C CNN
@@
 $EndComp
 $Comp
-L GND #PWR0105
+L GND #PWR315
 U 1 1 5723D1D2
 P 8200 1000
-F 0 "#PWR0105" H 8200 750 50  0001 C CNN
+F 0 "#PWR315" H 8200 750 50  0001 C CNN
 F 1 "GND" H 8200 850 50  0000 C CNN
 F 2 "" H 8200 1000 50  0000 C CNN
@@
 $EndComp
 $Comp
-L GND #PWR0106
+L GND #PWR317
 U 1 1 5723D249
 P 8500 1000
-F 0 "#PWR0106" H 8500 750 50  0001 C CNN
+F 0 "#PWR317" H 8500 750 50  0001 C CNN
 F 1 "GND" H 8500 850 50  0000 C CNN
 F 2 "" H 8500 1000 50  0000 C CNN
@@
 Wird UART benutzt?\nSystem Integration Manual  S.107
 NoConn ~ 4200 4650
+Text Notes 2450 2600 0    60   ~ 0
+So groß?
 $EndSCHEMATC

Commit message: sorted components
Connections:
- net RxD: no longer names the net of U301.17 (RXD)
- net TxD: no longer names the net of U301.16 (TXD)
- no-connect marks 27 -> 29
Changed lines of the file:
@@
 Wire Wire Line
 	2050 4800 2050 4900
-Text HLabel 3850 3350 0    60   Input ~ 0
-RxD
-Text HLabel 3850 3250 0    60   Input ~ 0
-TxD
 Wire Wire Line
 	3850 2950 4200 2950
 Wire Wire Line
 	3850 3050 4200 3050
-Wire Wire Line
-	3850 3250 4200 3250
-Wire Wire Line
-	3850 3350 4200 3350
 $Comp
 L R R303
@@
 Text Notes 2450 2600 0    60   ~ 0
 So groß?
+NoConn ~ 4200 3250
+NoConn ~ 4200 3350
 $EndSCHEMATC
