File: USB_HUB.sch (KiCad schematic (older format))
At the start: 26 parts, among them IC2 USB2514B, IC4 TPS2033, IC5 WE-TVS-82400274, IC6 WE-TVS-82400274, Y1 24M,18p

Commit message: added some footprints
Parts:
- C512: renamed from C12; footprint (none) -> Passives:C1206N
- renumbered C1 to C501, C2 to C502, C3 to C503, C4 to C504, C5 to C505, C8 to C506, C6 to C507, C7 to C508, C9 to C509, C10 to C510, C11 to C511, C13 to C513, C14 to C514, C15 to C515, IC2 to IC501, IC5 to IC502, IC4 to IC503, IC6 to IC504, R1 to R501, R2 to R502, R3 to R503, R4 to R504, R5 to R505, R6 to R506, Y1 to Y501
