File: power_supply.sch (KiCad schematic (older format))
At the start: 12 parts, among them IC704 TPS82085, IC705 TPS82085

Commit message: sorted components
Parts:
- C720, C721, C722, C723: footprint (none) -> Passives:C0805N
Connections:
- net GND: now also IC704.P, IC705.P
Changed lines of the file:
@@
 F 0 "C720" H 3300 2800 50  0000 L CNN
 F 1 "10u, 10V" H 3300 2600 50  0000 L CNN
-F 2 "" H 3288 2550 30  0001 C CNN
+F 2 "Passives:C0805N" H 3288 2550 30  0001 C CNN
 F 3 "" H 3300 2800 60  0000 C CNN
 	1    3250 2700
@@
 F 0 "C722" H 6700 2750 50  0000 L CNN
 F 1 "22u, 3mOhm" H 6700 2550 50  0000 L CNN
-F 2 "" H 6688 2500 30  0001 C CNN
+F 2 "Passives:C0805N" H 6688 2500 30  0001 C CNN
 F 3 "" H 6700 2750 60  0000 C CNN
 	1    6650 2650
@@
 Connection ~ 3750 2450
 $Comp
-L GND #PWR0143
+L GND #PWR702
 U 1 1 5729CB7E
 P 3250 3050
-F 0 "#PWR0143" H 3250 2800 50  0001 C CNN
+F 0 "#PWR702" H 3250 2800 50  0001 C CNN
 F 1 "GND" H 3250 2900 50  0000 C CNN
 F 2 "" H 3250 3050 50  0000 C CNN
@@
 $EndComp
 $Comp
-L GND #PWR0144
+L GND #PWR707
 U 1 1 5729CC25
 P 5850 3450
-F 0 "#PWR0144" H 5850 3200 50  0001 C CNN
+F 0 "#PWR707" H 5850 3200 50  0001 C CNN
 F 1 "GND" H 5850 3300 50  0000 C CNN
 F 2 "" H 5850 3450 50  0000 C CNN
@@
 	3250 2900 3250 3050
 $Comp
-L GND #PWR0145
+L GND #PWR705
 U 1 1 5729CEFC
 P 3950 3150
-F 0 "#PWR0145" H 3950 2900 50  0001 C CNN
+F 0 "#PWR705" H 3950 2900 50  0001 C CNN
 F 1 "GND" H 3950 3000 50  0000 C CNN
 F 2 "" H 3950 3150 50  0000 C CNN
@@
 $EndComp
 Wire Wire Line
-	3950 3150 3950 2900
+	3950 2800 3950 3150
 Wire Wire Line
 	3950 2900 4100 2900
@@
 Connection ~ 3950 3000
 $Comp
-L +5V #PWR0146
+L +5V #PWR701
 U 1 1 5729D450
 P 3250 2250
-F 0 "#PWR0146" H 3250 2100 50  0001 C CNN
+F 0 "#PWR701" H 3250 2100 50  0001 C CNN
 F 1 "+5V" H 3250 2390 50  0000 C CNN
 F 2 "" H 3250 2250 50  0000 C CNN
@@
 Connection ~ 3250 2350
 $Comp
-L GND #PWR0147
+L GND #PWR710
 U 1 1 5729DA4A
 P 6650 2950
-F 0 "#PWR0147" H 6650 2700 50  0001 C CNN
+F 0 "#PWR710" H 6650 2700 50  0001 C CNN
 F 1 "GND" H 6650 2800 50  0000 C CNN
 F 2 "" H 6650 2950 50  0000 C CNN
@@
 F 0 "C721" H 3400 4750 50  0000 L CNN
 F 1 "10u, 10V" H 3400 4550 50  0000 L CNN
-F 2 "" H 3388 4500 30  0001 C CNN
+F 2 "Passives:C0805N" H 3388 4500 30  0001 C CNN
 F 3 "" H 3400 4750 60  0000 C CNN
 	1    3350 4650
@@
 F 0 "C723" H 6800 4700 50  0000 L CNN
 F 1 "22u, 3mOhm" H 6800 4500 50  0000 L CNN
-F 2 "" H 6788 4450 30  0001 C CNN
+F 2 "Passives:C0805N" H 6788 4450 30  0001 C CNN
 F 3 "" H 6800 4700 60  0000 C CNN
 	1    6750 4600
@@
 Connection ~ 3850 4400
 $Comp
-L GND #PWR0148
+L GND #PWR704
 U 1 1 5729DE1A
 P 3350 5000
-F 0 "#PWR0148" H 3350 4750 50  0001 C CNN
+F 0 "#PWR704" H 3350 4750 50  0001 C CNN
 F 1 "GND" H 3350 4850 50  0000 C CNN
 F 2 "" H 3350 5000 50  0000 C CNN
@@
 $EndComp
 $Comp
-L GND #PWR0149
+L GND #PWR708
 U 1 1 5729DE20
 P 5950 5400
-F 0 "#PWR0149" H 5950 5150 50  0001 C CNN
+F 0 "#PWR708" H 5950 5150 50  0001 C CNN
 F 1 "GND" H 5950 5250 50  0000 C CNN
 F 2 "" H 5950 5400 50  0000 C CNN
@@
 	3350 4850 3350 5000
 $Comp
-L GND #PWR0150
+L GND #PWR706
 U 1 1 5729DE28
 P 4050 5100
-F 0 "#PWR0150" H 4050 4850 50  0001 C CNN
+F 0 "#PWR706" H 4050 4850 50  0001 C CNN
 F 1 "GND" H 4050 4950 50  0000 C CNN
 F 2 "" H 4050 5100 50  0000 C CNN
@@
 $EndComp
 Wire Wire Line
-	4050 5100 4050 4850
+	4050 4750 4050 5100
 Wire Wire Line
 	4050 4850 4200 4850
@@
 Connection ~ 4050 4950
 $Comp
-L +5V #PWR0151
+L +5V #PWR703
 U 1 1 5729DE32
 P 3350 4200
-F 0 "#PWR0151" H 3350 4050 50  0001 C CNN
+F 0 "#PWR703" H 3350 4050 50  0001 C CNN
 F 1 "+5V" H 3350 4340 50  0000 C CNN
 F 2 "" H 3350 4200 50  0000 C CNN
@@
 Connection ~ 3350 4300
 $Comp
-L GND #PWR0152
+L GND #PWR712
 U 1 1 5729DE39
 P 6750 4900
-F 0 "#PWR0152" H 6750 4650 50  0001 C CNN
+F 0 "#PWR712" H 6750 4650 50  0001 C CNN
 F 1 "GND" H 6750 4750 50  0000 C CNN
 F 2 "" H 6750 4900 50  0000 C CNN
@@
 	6750 4800 6750 4900
 $Comp
-L +3V8 #PWR0153
+L +3V8 #PWR711
 U 1 1 5729D386
 P 6750 4150
-F 0 "#PWR0153" H 6750 4000 50  0001 C CNN
+F 0 "#PWR711" H 6750 4000 50  0001 C CNN
 F 1 "+3V8" H 6750 4290 50  0000 C CNN
 F 2 "" H 6750 4150 50  0000 C CNN
@@
 Connection ~ 6750 4300
 $Comp
-L +3.3V #PWR0154
+L +3.3V #PWR709
 U 1 1 5729D7D3
 P 6650 2200
-F 0 "#PWR0154" H 6650 2050 50  0001 C CNN
+F 0 "#PWR709" H 6650 2050 50  0001 C CNN
 F 1 "+3.3V" H 6650 2340 50  0000 C CNN
 F 2 "" H 6650 2200 50  0000 C CNN
@@
 	1    0    0    -1
 $EndComp
+Wire Wire Line
+	3950 2800 4100 2800
+Connection ~ 3950 2900
+Wire Wire Line
+	4200 4750 4050 4750
+Connection ~ 4050 4850
 $EndSCHEMATC

Commit message: power Sypply for Tobyfinish
Other:
- moved on the sheet: C721, C723, IC705, R717, R718, R720
