File: tinyLinuxModuleVybrid.kicad_pcb (KiCad board)
At the start: 4 copper layers, 91.4 x 48.3 mm, 185 parts, among them IC201 LAN8720, IC401 WM-294, IC501 USB2514B, IC502 WE-TVS-82400274, IC503 TPS2033, IC504 WE-TVS-82400274, IC704 TPS82085, IC705 TPS82085, IC801 BME680, M102 SCREW, M104 SCREW, M106 SCREW, M108 SCREW, Q101 2N7002BKT, Q102 2N7002BKT, Q103 2N7002BKT, Q301 2N7002BKT, Q601 2N7002BKT, U301 U-BLOX-TOBY-L2, U401 U-BLOX_LILY-W1, U601 U-BLOX-NEO-M8N, U801 MPU-9250, U802 LMT86, X101 MICROSD, X102 LAN_Transformer, X103 CONN_01x06, X104 VybridBoard, X105 ARM_JTAG_10, X301 ANT, X302 SIMcard, X303 ANT, X401 ANT, X601 ANT, Y501 24M,18p

Commit message: Toby Antenne und Simkarte gerootet
Parts:
- moved M108 14.3 mm to (250.2, 88.5)
- moved C721 14.3 mm to (222.8, 117.7)
- moved IC705 14.3 mm to (222.8, 120.5)
- moved R717 14.3 mm to (223.6, 123.5)
- moved R718 14.3 mm to (222.3, 123.5)
- moved C723 14.3 mm to (225.6, 120.5)
- moved R720 13.9 mm to (220.7, 122.8)
- moved D305 10.8 mm to (214.1, 103.5), turned to 180 degrees
- moved D302 10.2 mm to (210.7, 101.0), turned to 270 degrees
- moved D303 8.41 mm to (209.4, 100.8), turned to 270 degrees
- moved D301 8.29 mm to (206.1, 97.7), turned to 270 degrees
- moved D304 5.93 mm to (208.1, 100.9), turned to 270 degrees
- moved R306 2.03 mm to (229.8, 118.2)
- moved C301 1.73 mm to (224.3, 119.3)
- moved C305 0.71 mm to (224.3, 120.5)
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Routing:
- net Net-(C311-Pad1): track 0.00 -> 15.9 mm, vias 0 -> 1
- net Net-(C308-Pad1): track 0.00 -> 15.6 mm, vias 0 -> 1
- net Net-(C309-Pad1): track 0.00 -> 15.3 mm, vias 0 -> 1
- net Net-(C312-Pad2): track 0.00 -> 14.9 mm, vias 0 -> 2
- net Net-(C313-Pad1): track 0.00 -> 11.4 mm, vias 0 -> 1
- net Net-(IC705-Pad7): track 0.00 -> 11.3 mm
- net Net-(LED301-PadC): track 0.00 -> 4.24 mm
- net Net-(C314-Pad1): track 0.00 -> 2.81 mm
- net Net-(C310-Pad1): track 0.00 -> 2.79 mm
- net Net-(R302-Pad1): track 0.00 -> 2.30 mm
- net Net-(R306-Pad2): track 0.00 -> 2.21 mm
- net Net-(R303-Pad1): track 0.00 -> 2.01 mm
- net Net-(R304-Pad1): track 0.00 -> 1.95 mm
- net Net-(R307-Pad2): track 0.00 -> 1.89 mm
- net Net-(R305-Pad2): track 0.00 -> 1.88 mm
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- added copper zone on B.Cu, net +3V8
- added copper zone on F.Cu, net +3V8
- added copper zone on B.Cu, net +5V
- added copper zone on B.Cu, net GND
- added copper zone on F.Cu, net GND
- added copper zone on F.Cu, net Net-(C312-Pad2)
- added copper zone on B.Cu, net Net-(C313-Pad1)

Commit message: power Sypply for Tobyfinish
Parts:
- removed IC401: WM-294, Communication:WM-294
- C103, C104, C201, C202, C204, C205, C207, C208, C209, C210, IC201, L201, R201, R202, R203, R204, R205, R206, R207, R208, R209, R210, R211, X103: moved to B.Cu
- moved C201 78.2 mm to (184.4, 109.3), turned to 90 degrees
- moved C202 76.4 mm to (188.5, 109.3), turned to 90 degrees
- moved C204 66.8 mm to (183.9, 111.4)
- moved C205 65.3 mm to (190.6, 112.9), turned to 180 degrees
- moved C210 63.6 mm to (189.1, 106.9)
- moved C207 63.1 mm to (184.9, 106.9)
- moved X104 46.8 mm to (117.1, 134.3)
- moved C602 24.7 mm to (207.7, 148.7)
- moved R602 24.7 mm to (207.7, 151.0)
- moved R604 24.7 mm to (207.7, 149.7)
- moved C601 24.7 mm to (207.7, 147.7)
- moved R606 22.5 mm to (191.4, 155.9)
- moved L601 22.4 mm to (201.6, 155.8)
- moved X601 22.4 mm to (202.1, 159.1)
- moved U601 22.4 mm to (196.2, 147.7)
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Connections:
- net /Communication/NEO/RX renamed /Communication/RX_NEO
- net /Communication/NEO/TX renamed /Communication/TX_NEO
- net /Communication/TOBY/RxD renamed Net-(U301-Pad17)
- net /Communication/TOBY/TxD renamed Net-(U301-Pad16)
- net /PTA6 renamed /Communication/RMII_REFCLK
- net /PTC10 renamed /Communication/RMII_MDIO
- net /PTC11 renamed /Communication/RMII_CRSDV
- net /PTC12 renamed /Communication/RMII_RX1
- net /PTC13 renamed /Communication/RMII_RX0
- net /PTC14 renamed /Communication/RMII_RXER
- net /PTC15 renamed /Communication/RMII_TX1
- net /PTC16 renamed /Communication/RMII_TX0
- net /PTC17 renamed /Communication/RMII_TXEN
- net /PTC9 renamed /Communication/RMII_MDC
- net /USB0_D_N renamed /Communication/USB_D-
- net /USB0_D_P renamed /Communication/USB_D+
- C514 pad 1: /Communication/USB_HUB/USB_VBUS_OUT -> /Communication/USB_VBUS_OUT
- C515 pad 1: /Communication/USB_HUB/USB_VBUS_OUT -> /Communication/USB_VBUS_OUT
- D301 pad A: /~RESET -> /Communication/~RESET
- IC201 pad 15: /~RESET -> /Communication/~RESET
- IC501 pad 13: /Communication/USB_HUB/USB_VBUS_OC -> /Communication/USB_VBUS_OC
- IC501 pad 17: /Communication/USB_HUB/USB_VBUS_OC -> /Communication/USB_VBUS_OC
- IC501 pad 19: /Communication/USB_HUB/USB_VBUS_OC -> /Communication/USB_VBUS_OC
- IC501 pad 21: /Communication/USB_HUB/USB_VBUS_OC -> /Communication/USB_VBUS_OC
- IC501 pad 26: /Communication/USB_HUB/~RESET -> /Communication/~RESET
- IC502 pad 5: /Communication/USB_HUB/USB_VBUS_OUT -> /Communication/USB_VBUS_OUT
- IC503 pad 4: /Communication/USB_HUB/USB_VBUS_EN -> /Communication/USB_VBUS_EN
- IC503 pad 5: /Communication/USB_HUB/USB_VBUS_OC -> /Communication/USB_VBUS_OC
- IC503 pad 6: /Communication/USB_HUB/USB_VBUS_OUT -> /Communication/USB_VBUS_OUT
- IC503 pad 7: /Communication/USB_HUB/USB_VBUS_OUT -> /Communication/USB_VBUS_OUT
- IC503 pad 8: /Communication/USB_HUB/USB_VBUS_OUT -> /Communication/USB_VBUS_OUT
- IC504 pad 5: /Communication/USB_HUB/USB_VBUS_OUT -> /Communication/USB_VBUS_OUT
- R506 pad 2: /Communication/USB_HUB/USB_VBUS_OC -> /Communication/USB_VBUS_OC
- U301 pad 23: /~RESET -> /Communication/~RESET
- U401 pad 8: +3V3 -> Net-(U401-Pad8)
- U601 pad 8: /Communication/NEO/~RESET -> /Communication/~RESET
- X104 pad 190: /~RESET -> /Communication/~RESET
- X104 pad 74: /PTA17 -> /Communication/USB_VBUS_OC
- X104 pad 75: /USB0_VBUS -> /Communication/USB_VBUS_OUT
- X104 pad 76: /PTA16 -> /Communication/USB_VBUS_EN
- X105 pad 10: /~RESET -> /Communication/~RESET
Routing:
- net /Communication/USB_HUB/USBB_D+: track 0.00 -> 20.7 mm
- net /Communication/USB_HUB/USBB_D-: track 0.00 -> 19.3 mm
- net /Communication/ETH_TX-: track 0.00 -> 15.1 mm, vias 0 -> 2
- net /Communication/ETH_TX+: track 0.00 -> 13.9 mm
- net Net-(C204-Pad2): track 0.00 -> 10.4 mm
- net +3V8: track 0.00 -> 9.91 mm, vias 0 -> 1
- net (no net): track 279.4 -> 288.4 mm, vias 0 -> 36
- net Net-(D101-PadA): track 0.00 -> 8.30 mm
- net Net-(X102-Pad16): track 0.00 -> 8.20 mm
- net GND: track 0.00 -> 5.90 mm, vias 0 -> 5
- net +5V: track 0.00 -> 4.54 mm, vias 0 -> 2
- net Net-(IC201-Pad2): track 1.51 -> 5.63 mm
- net Net-(L601-Pad1): track 0.00 -> 4.02 mm
- net Net-(IC201-Pad3): track 1.84 -> 5.73 mm
- net Net-(IC705-Pad2): track 0.00 -> 2.78 mm
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- added copper zone on F.Cu, net +3V3
Other:
- copper layers 4 -> 6

Commit message: stecker hinzugefügt
Parts:
- removed D101: DP, Passives:D_0402
- removed G***: LOGO, Symbols:hsrm_logo
- removed R116, R117: Anpassen, Passives:R0402N
- removed R118, R119, R120, R121: 75, Passives:R0402N
- removed REF**: Symbol_ESD-Logo_CopperTop, Symbols:Symbol_ESD-Logo_CopperTop
- added X106: CONN_02x50, Connector:ERF8-50-05.0-L-DV-K-TR, B.Cu at (177.7, 134.9)
- C207, C210, R208, R211: moved to F.Cu
- C211, C406: moved to B.Cu
- moved M104 126.4 mm to (143.4, 134.4)
- moved M102 122.1 mm to (143.5, 94.4)
- moved C203 67.5 mm to (192.5, 117.0)
- moved C206 61.3 mm to (192.4, 115.2)
- moved C211 58.9 mm to (189.8, 115.7), turned to 180 degrees
- moved X104 51.3 mm to (162.6, 110.7)
- moved C101 38.4 mm to (163.2, 107.6)
- moved C102 38.4 mm to (163.1, 105.0)
- moved X105 36.4 mm to (143.2, 110.8), turned to 180 degrees
- moved R101 35.4 mm to (160.9, 124.3)
- moved R102 35.4 mm to (162.4, 124.3)
- moved R103 35.4 mm to (163.9, 124.3)
- moved R104 35.4 mm to (165.5, 124.3)
- moved R105 35.4 mm to (167.0, 124.3)
- moved R106 35.4 mm to (168.5, 124.3)
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Connections:
- net /Communication/RMII_CRSDV renamed /PTC11
- net /Communication/RMII_MDC renamed /PTC9
- net /Communication/RMII_MDIO renamed /PTC10
- net /Communication/RMII_REFCLK renamed /PTA6
- net /Communication/RMII_RX0 renamed /PTC13
- net /Communication/RMII_RX1 renamed /PTC12
- net /Communication/RMII_RXER renamed /PTC14
- net /Communication/RMII_TX0 renamed /PTC16
- net /Communication/RMII_TX1 renamed /PTC15
- net /Communication/RMII_TXEN renamed /PTC17
- net /Communication/USB_D+ renamed /USB0_D_P
- net /Communication/USB_D- renamed /USB0_D_N
- net /Communication/USB_VBUS_EN renamed /PTA16
- net /Communication/USB_VBUS_OC renamed /PTA17
- net /Communication/USB_VBUS_OUT renamed /USB0_VBUS
- net /Communication/~RESET renamed /~RESET
- IC201 pad 4: Net-(IC201-Pad4) -> (no net)
- IC501 pad 12: Net-(IC501-Pad12) -> (no net)
- IC501 pad 16: Net-(IC501-Pad16) -> (no net)
- IC501 pad 18: Net-(IC501-Pad18) -> (no net)
- IC501 pad 20: Net-(IC501-Pad20) -> (no net)
- IC503 pad 3: Net-(IC503-Pad3) -> (no net)
- IC801 pad 5: /Sensors/SDO -> (no net)
- LED104 pad A: Net-(LED104-PadA) -> /Communication/ETH_LED_SPD-
- LED105 pad A: Net-(LED105-PadA) -> /Communication/ETH_LED_ACT+
- R602 pad 2: /Communication/RX_NEO -> (no net)
- R604 pad 2: /Communication/TX_NEO -> (no net)
- U301 pad 10: Net-(U301-Pad10) -> (no net)
- U301 pad 11: Net-(U301-Pad11) -> (no net)
- U301 pad 12: Net-(U301-Pad12) -> (no net)
- U301 pad 15: Net-(U301-Pad15) -> (no net)
- U301 pad 16: Net-(U301-Pad16) -> (no net)
- U301 pad 17: Net-(U301-Pad17) -> (no net)
- U301 pad 20: /Communication/TOBY/PWR_ON -> (no net)
- U301 pad 22: Net-(U301-Pad22) -> (no net)
- U301 pad 24: Net-(U301-Pad24) -> (no net)
- U301 pad 25: Net-(U301-Pad25) -> (no net)
- U301 pad 26: Net-(U301-Pad26) -> (no net)
- U301 pad 3: Net-(C307-Pad+) -> (no net)
- U301 pad 4: Net-(U301-Pad4) -> (no net)
- U301 pad 5: +1V8 -> (no net)
- U301 pad 50: Net-(U301-Pad50) -> (no net)
- U301 pad 51: Net-(U301-Pad51) -> (no net)
- U301 pad 52: Net-(U301-Pad52) -> (no net)
- U301 pad 53: Net-(U301-Pad53) -> (no net)
- U301 pad 54: Net-(U301-Pad54) -> (no net)
- U301 pad 55: Net-(U301-Pad55) -> (no net)
- U301 pad 60: Net-(U301-Pad60) -> (no net)
- U301 pad 61: Net-(U301-Pad61) -> (no net)
- U301 pad 62: Net-(U301-Pad62) -> (no net)
- U301 pad 63: Net-(U301-Pad63) -> (no net)
- U301 pad 64: Net-(U301-Pad64) -> (no net)
- U301 pad 65: Net-(U301-Pad65) -> (no net)
- U301 pad 66: Net-(U301-Pad66) -> (no net)
- U301 pad 67: Net-(U301-Pad67) -> (no net)
- U301 pad 68: Net-(U301-Pad68) -> (no net)
- U401 pad 1: Net-(U401-Pad1) -> (no net)
- U401 pad 14: /Communication/LILY/POWER_DOWN-N -> (no net)
- U401 pad 15: Net-(U401-Pad15) -> (no net)
- U401 pad 16: Net-(U401-Pad16) -> (no net)
- U401 pad 17: /Communication/LILY/WAKE_UP -> (no net)
- U401 pad 18: Net-(U401-Pad18) -> (no net)
- U401 pad 19: /Communication/LILY/HOST_WKUP -> (no net)
- U401 pad 2: Net-(U401-Pad2) -> (no net)
- U401 pad 20: Net-(U401-Pad20) -> (no net)
- U401 pad 22: Net-(U401-Pad22) -> (no net)
- U401 pad 3: Net-(U401-Pad3) -> (no net)
- U401 pad 5: Net-(U401-Pad5) -> (no net)
- U401 pad 7: Net-(U401-Pad7) -> (no net)
- U401 pad 8: Net-(U401-Pad8) -> +3V3
- U601 pad 1: Net-(U601-Pad1) -> (no net)
- U601 pad 15: Net-(U601-Pad15) -> (no net)
- U601 pad 16: Net-(U601-Pad16) -> (no net)
- U601 pad 17: Net-(U601-Pad17) -> (no net)
- U601 pad 18: Net-(U601-Pad18) -> (no net)
- U601 pad 19: Net-(U601-Pad19) -> (no net)
- U601 pad 2: Net-(U601-Pad2) -> (no net)
- U601 pad 4: Net-(U601-Pad4) -> (no net)
- U601 pad 5: Net-(U601-Pad5) -> (no net)
- U601 pad 6: Net-(U601-Pad6) -> (no net)
- U801 pad 1: Net-(U801-Pad1) -> (no net)
- U801 pad 12: /Sensors/INT -> (no net)
- U801 pad 14: Net-(U801-Pad14) -> (no net)
- U801 pad 17: Net-(U801-Pad17) -> (no net)
- U801 pad 19: Net-(U801-Pad19) -> (no net)
- U801 pad 2: Net-(U801-Pad2) -> (no net)
- U801 pad 21: Net-(U801-Pad21) -> (no net)
- U801 pad 22: /Sensors/~CS -> (no net)
- U801 pad 23: /Sensors/SCL -> (no net)
- U801 pad 24: /Sensors/SDA -> (no net)
- U801 pad 3: Net-(U801-Pad3) -> (no net)
- U801 pad 4: Net-(U801-Pad4) -> (no net)
- U801 pad 5: Net-(U801-Pad5) -> (no net)
- U801 pad 6: Net-(U801-Pad6) -> (no net)
- U801 pad 7: Net-(U801-Pad7) -> (no net)
- U801 pad 9: Net-(U801-Pad9) -> (no net)
- U802 pad 3: /Sensors/TEMP_SENSOR -> /ADC0SE9
- X102 pad 10: Net-(R119-Pad2) -> GND
- X102 pad 15: Net-(R118-Pad2) -> GND
- X103 pad 1: Net-(X102-Pad9) -> Net-(X102-Pad16)
- X103 pad 2: Net-(R121-Pad1) -> GND
- X103 pad 3: Net-(X102-Pad11) -> Net-(X102-Pad14)
- X103 pad 4: Net-(X102-Pad14) -> Net-(X102-Pad11)
- X103 pad 5: Net-(R120-Pad1) -> GND
- X103 pad 6: Net-(X102-Pad16) -> Net-(X102-Pad9)
- X104 pad 100: /ADC1SE9 -> (no net)
- X104 pad 101: /PTA20 -> (no net)
- X104 pad 102: /PTA23 -> (no net)
- X104 pad 103: /PTB14 -> (no net)
- X104 pad 104: /PTE20 -> (no net)
- X104 pad 105: /PTB17 -> (no net)
- X104 pad 106: /PTB18 -> (no net)
- X104 pad 107: /PTB10 -> (no net)
- X104 pad 108: /PTB20 -> (no net)
- X104 pad 109: /PTB28 -> (no net)
- X104 pad 110: /PTB15 -> (no net)
- X104 pad 113: /PTB23 -> (no net)
- X104 pad 114: /PTB25 -> (no net)
- X104 pad 115: /PTE27 -> (no net)
- X104 pad 116: /PTB26 -> (no net)
- X104 pad 117: /PTE25 -> (no net)
- X104 pad 118: /PTC29 -> (no net)
- X104 pad 119: /PTE26 -> (no net)
- X104 pad 120: /PTB24 -> (no net)
- X104 pad 123: /PTB19 -> (no net)
- X104 pad 124: /PTA21 -> (no net)
- X104 pad 125: /PTD18 -> (no net)
- X104 pad 126: /PTD16 -> (no net)
- X104 pad 127: /PTC26 -> (no net)
- X104 pad 128: /PTE24 -> (no net)
- X104 pad 129: /PTD20 -> (no net)
- X104 pad 130: /PTD17 -> (no net)
- X104 pad 133: /PTD25 -> (no net)
- X104 pad 135: /PTD29 -> (no net)
- X104 pad 137: /PTE23 -> (no net)
- X104 pad 139: /PTB8 -> (no net)
- X104 pad 14: /PTA12 -> (no net)
- X104 pad 140: /PTD24 -> (no net)
- X104 pad 143: /PTE12 -> (no net)
- X104 pad 144: /PTD30 -> (no net)
- X104 pad 145: /PTE15 -> (no net)
- X104 pad 146: /PTB9 -> (no net)
- X104 pad 147: /PTE9 -> (no net)
- X104 pad 148: /PTD31 -> (no net)
- X104 pad 149: /PTD26 -> (no net)
- X104 pad 150: /PTE18 -> (no net)
- X104 pad 153: /PTB21 -> (no net)
- X104 pad 154: /PTE17 -> (no net)
- X104 pad 155: /PTB7 -> (no net)
- X104 pad 156: /PTE19 -> (no net)
- X104 pad 157: /PTB12 -> (no net)
- X104 pad 158: /PTE16 -> (no net)
- X104 pad 159: /PTC28 -> (no net)
- X104 pad 160: /PTE8 -> (no net)
- X104 pad 163: /PTC27 -> (no net)
- X104 pad 164: /PTE7 -> (no net)
- X104 pad 165: /PTB11 -> (no net)
- X104 pad 166: /PTE2 -> (no net)
- X104 pad 167: /PTB16 -> (no net)
- X104 pad 168: /PTE4 -> (no net)
- X104 pad 169: /PTB22 -> (no net)
- X104 pad 170: /PTE1 -> (no net)
- X104 pad 173: /PTD19 -> (no net)
- X104 pad 174: /PTA22 -> (no net)
- X104 pad 175: /PTD28 -> (no net)
- X104 pad 176: /PTB13 -> (no net)
- X104 pad 177: /PTD27 -> (no net)
- X104 pad 178: /PTE14 -> (no net)
- X104 pad 179: /PTE28 -> (no net)
- X104 pad 18: /PTC7 -> (no net)
- X104 pad 180: /PTE3 -> (no net)
- X104 pad 183: /PTE11 -> (no net)
- X104 pad 184: /PTE0 -> (no net)
- X104 pad 185: /PTE22 -> (no net)
- X104 pad 186: /PTE5 -> (no net)
- X104 pad 187: /PTE6 -> (no net)
- X104 pad 188: /VBAT -> (no net)
- X104 pad 189: /PTE13 -> (no net)
- X104 pad 193: /PTD13 -> (no net)
- X104 pad 195: /PTD8 -> (no net)
- X104 pad 197: /PTE10 -> (no net)
- X104 pad 199: /PTE21 -> (no net)
- X104 pad 28: /PTB0 -> (no net)
- X104 pad 30: /PTB1 -> (no net)
- X104 pad 34: /PTC30 -> (no net)
- X104 pad 36: /PTD12 -> (no net)
- X104 pad 38: /PTD4 -> (no net)
- X104 pad 39: /PTD7 -> (no net)
- X104 pad 40: /PTD5 -> (no net)
- X104 pad 44: /PTD6 -> (no net)
- X104 pad 45: /PTA7 -> (no net)
- X104 pad 46: /PTD10 -> (no net)
- X104 pad 48: /PTD11 -> (no net)
- X104 pad 49: /PTD0 -> (no net)
- X104 pad 50: /PTD1 -> (no net)
- X104 pad 51: /PTD3 -> (no net)
- X104 pad 53: /PTD9 -> (no net)
- X104 pad 54: /PTC8 -> (no net)
- X104 pad 55: /PTD2 -> (no net)
- X104 pad 59: /PTA30 -> (no net)
- X104 pad 60: /PTA19 -> (no net)
- X104 pad 61: /PTA31 -> (no net)
- X104 pad 64: /PTA18 -> (no net)
- X104 pad 66: /PTB2 -> (no net)
- X104 pad 68: /PTB27 -> (no net)
- X104 pad 70: /PTC31 -> (no net)
- X104 pad 77: /USB1_VBUS -> (no net)
- X104 pad 78: /PTB3 -> (no net)
- X104 pad 80: /PTB4 -> (no net)
- X104 pad 81: /USB1_D+ -> (no net)
- X104 pad 83: /USB1_D- -> (no net)
- X104 pad 84: /PTB6 -> (no net)
- X104 pad 86: /PTB5 -> (no net)
- X104 pad 88: /DAC0 -> (no net)
- X104 pad 90: /DAC1 -> (no net)
- X104 pad 93: /VADCSE2 -> (no net)
- X104 pad 95: /VADCSE0 -> (no net)
- X104 pad 96: /ADC0SE8 -> (no net)
- X104 pad 97: /VADCSE1 -> (no net)
- X104 pad 98: /ADC1SE8 -> (no net)
- X104 pad 99: /VADCSE3 -> (no net)
- X105 pad 7: Net-(X105-Pad7) -> (no net)
- X105 pad 9: Net-(X105-Pad9) -> (no net)
Routing:
- net /Communication/USB_HUB/USBB_D+: track 20.7 -> 0.00 mm
- net /Communication/USB_HUB/USBB_D-: track 19.3 -> 0.00 mm
- net GND: track 5.90 -> 19.5 mm, vias 5 -> 22
- net /Communication/ETH_RX-: track 0.00 -> 9.78 mm, vias 0 -> 1
- net +3V3: track 2.09 -> 11.1 mm, vias 2 -> 10
- net Net-(D101-PadA): track 8.30 -> 0.00 mm
- net /Communication/ETH_TX-: track 15.1 -> 7.34 mm, vias 2 -> 1
- net /Communication/ETH_RX+: track 0.00 -> 6.98 mm, vias 0 -> 1
- net Net-(X102-Pad16): track 8.20 -> 2.59 mm, vias 0 -> 1
- net /Communication/ETH_TX+: track 13.9 -> 9.74 mm, vias 0 -> 1
- net Net-(L601-Pad1): track 4.02 -> 0.00 mm
- net Net-(IC201-Pad2): track 5.63 -> 1.91 mm
- net Net-(IC201-Pad3): track 5.73 -> 2.51 mm
- net Net-(C204-Pad2): track 10.4 -> 7.33 mm
- net Net-(X102-Pad11): track 0.00 -> 2.83 mm, vias 0 -> 1
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- added copper zone on B.Cu, net +3V3
- added copper zone on GND.Cu, net GND
Other:
- board size 91.4 x 48.3 mm -> 102.1 x 48.3 mm

Commit message: sd card
Parts:
- moved C501 98.2 mm to (166.2, 146.3)
- moved C502 98.2 mm to (166.0, 159.1)
- moved C503 98.2 mm to (164.5, 154.2)
- moved C504 98.2 mm to (160.4, 164.6)
- moved C505 98.2 mm to (159.6, 154.5)
- moved C507 98.2 mm to (161.7, 146.3)
- moved C509 98.2 mm to (157.4, 160.3)
- moved C513 98.2 mm to (178.4, 169.5)
- moved IC502 98.2 mm to (168.8, 156.5)
- moved IC503 98.2 mm to (170.6, 167.7)
- moved R503 98.2 mm to (158.9, 151.7)
- moved R504 98.2 mm to (157.9, 164.6)
- moved R505 98.2 mm to (163.2, 154.2)
- moved R506 98.2 mm to (164.5, 164.9)
- moved Y501 98.2 mm to (162.7, 149.4)
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Routing:
- net /PTC2: track 0.00 -> 31.4 mm, vias 0 -> 1
- net /PTC4: track 0.00 -> 31.1 mm, vias 0 -> 2
- net /PTC5: track 0.00 -> 31.1 mm, vias 0 -> 2
- net /PTC0: track 0.00 -> 31.0 mm, vias 0 -> 2
- net /PTC3: track 0.00 -> 31.0 mm, vias 0 -> 2
- net /PTC1: track 0.00 -> 30.9 mm, vias 0 -> 1
- net GND: track 19.5 -> 36.3 mm, vias 22 -> 24
- net /PTC6: track 0.00 -> 15.4 mm, vias 0 -> 1
- net +3V3: track 11.1 -> 24.8 mm, vias 10 -> 12
- net (no net): vias 1 -> 0
- added copper zone on VCC.Cu, net +3V3
Other:
- board size 102.1 x 48.3 mm -> 105.3 x 50.8 mm
